File: pinkman/pinkman.kicad_sch (KiCad schematic)
At the start: 1 part, among them J1 TSM-110-01-T-DV

Commit message: Update pinkman.kicad_sch
Parts:
- added C1: 100 nF, symbol Device:C
- added U1: LPS22DFTR, QFN_22DFTR_STM, symbol Pinkman Altimeter:LPS22DFTR
Connections:
- net DIGI_BARO_DRDY_L: now reaches J1.12
- net DIGI_BARO_DRDY_L: now also U1.7 (INT_DRDY)
- net DIGI_BARO_SCL_H: now reaches J1.14
- net DIGI_BARO_SDA_H: now reaches J1.16
- net DIGI_BARO_SDA_H: now also U1.4 (SDA/SDI/SDISDO)
- new net: C1.2, U1.1 (Vdd_IO), U1.10 (VDD)
- new net Earth: C1.1, U1.3 (RES), U1.5 (SDO/SA0), U1.6 (CS), U1.8 (GND_IO), U1.9 (GND)

Commit message: added symbols and ground
Parts:
- added GPS: MAX-M10M-00B, MOD18_MAX-M10M_UBL, symbol GPS:MAX-M10M-00B
- added IMU: LSM6DSO32TR, LGA-14L_2P5X3X0P83_STM, symbol IMU:LSM6DSO32TR
- added Radio: RA-02, RA-02_AIT, symbol Radio:RA-02
- added Regulator: LTC3601EMSE-TRPBF, MSOP-16_MSE_LIT, symbol Regulator:LTC3601EMSE-TRPBF
- renumbered U1 to Altimeter
Connections:
- net Earth: now also J1.1, GPS.1 (GND), GPS.10 (GND), GPS.12 (GND), IMU.6 (GND), IMU.7 (GND), Radio.1 (GND), Radio.16 (GND), Radio.2 (GND), Radio.9 (GND), Regulator.3 (PGND), Regulator.4 (PGND)
