File: pinkman/pinkman.kicad_sch (KiCad schematic)
At the start: 3 parts, among them J1 TSM-110-01-T-DV, U1 LPS22DFTR

Commit message: Finished Schematic
Used AI to help me with schematic design. Added a second page for Power & GNSS support.
Parts:
- removed J1: TSM-110-01-T-DV, MDFC Common:CONN_TSM-110-01-T-DV_SAI, symbol MDFC Common:TSM-110-01-T-DV
- removed U1: LPS22DFTR, QFN_22DFTR_STM, symbol Pinkman Altimeter:LPS22DFTR
- added C2, C3, C4, C5, C6, C8: 100nF, Capacitor_SMD:C_0603_1608Metric, symbol Device:C
- added C7, C9: 10uF, Capacitor_SMD:C_0805_2012Metric, symbol Device:C
- added J1: TSM-110-01-T-DV, MDFC Common:CONN_TSM-110-01-T-DV_SAI, symbol Connector_Generic:Conn_02x10_Odd_Even
- added R1, R2: 4.7k, Resistor_SMD:R_0603_1608Metric, symbol Device:R
- added R3, R4: 10k, Resistor_SMD:R_0603_1608Metric, symbol Device:R
- added TP1: IMU_INT1, TestPoint:TestPoint_Pad_D1.5mm, symbol Connector:TestPoint
- added U1: LPS22DFTR, Pinkman Local:QFN_22DFTR_STM, symbol Pinkman Local:LPS22DFTR
- added U2: LSM6DSO32TR, Pinkman Local:LGA-14L_2P5X3X0P83_STM, symbol Pinkman Local:LSM6DSO32TR
- added U3: MAX-M10M-00B, Pinkman Local:MOD18_MAX-M10M_UBL, symbol Pinkman Local:MAX-M10M-00B
- added U4: RA-02, Pinkman Local:RA-02_AIT, symbol Pinkman Local:RA-02
- added U5: LTC3601EMSE-TRPBF, Pinkman Local:MSOP-16_MSE_LIT, symbol Pinkman Local:LTC3601EMSE-TRPBF
- C1: value 100 nF -> 100nF; footprint (none) -> Capacitor_SMD:C_0603_1608Metric
Connections:
- net GND: now reaches C1.2
- net GND: now also C2.2, C3.2, C4.2, C5.2, C6.2, C7.2, C8.2, C9.2, J1.1 (Pin_1), J1.2 (Pin_2), J1.3 (Pin_3), J1.4 (Pin_4), U1.3 (RES), U1.5 (SDO/SA0), U1.8 (GND_IO), U1.9 (GND), U2.1 (SDO/SA0), U2.2 (SDx), U2.3 (SCx), U2.6 (GND), U2.7 (GND), U3.1 (GND), U3.10 (GND), U3.12 (GND), U4.1 (GND), U4.16 (GND), U4.2 (GND), U4.9 (GND), U5.15 (MODE/SYNC), U5.17 (EPAD), U5.3 (PGND), U5.4 (PGND)
- net Earth renamed +3V3
- net +3V3: now also C2.1, C3.1, C4.1, C5.1, C6.1, C7.1, C8.1, C9.1, R1.1, R2.1, R3.1, R4.1, U1.1 (Vdd_IO), U1.10 (VDD), U1.6 (CS), U2.12 (CS), U2.5 (VDDIO), U2.8 (VDD), U3.7 (V_IO), U3.8 (VCC), U4.3 (3.3V), U5.7 (VON)
- new net +5V_IN: J1.7 (Pin_7), U5.12 (RUN), U5.13 (VIN), U5.14 (VIN)
- new net BARO_DRDY: J1.20 (Pin_20), U1.7 (INT_DRDY)
- new net BOOST: U5.5 (BOOST)
- new net FB: U5.9 (FB)
- new net GNSS_RF: U3.11 (RF_IN)
- new net GPS_PPS: J1.14 (Pin_14), U3.4 (TIMEPULSE)
- new net GPS_VCC_RF: U3.14 (VCC_RF)
- new net HOST_UART_RX: J1.18 (Pin_18), U3.2 (TXD)
- new net HOST_UART_TX: J1.16 (Pin_16), U3.3 (RXD)
- new net I2C_SCL: J1.6 (Pin_6), R2.2, U1.2 (SCL), U2.13 (SCL), U3.17 (SCL)
- new net I2C_SDA: J1.8 (Pin_8), R1.2, U1.4 (SDA/SDI/SDISDO), U2.14 (SDA), U3.16 (SDA)
- new net IMU_INT1: TP1.1, U2.4 (INT1)
- new net INTVCC: U5.10 (ITH), U5.6 (INTVCC), U5.8 (RT)
- new net POWER_GOOD: U5.16 (PGOOD)
- new net RADIO_DIO0: J1.15 (Pin_15), U4.5 (DIO0)
- new net RADIO_DIO1: J1.12 (Pin_12), U4.6 (DIO1)
- new net RADIO_RESET_N: J1.9 (Pin_9), R3.2, U4.4 (RESET)
- new net SOFTSTART: U5.11 (TRACK)
- new net SPI_CS_N: J1.11 (Pin_11), R4.2, U4.15 (NSS)
- new net SPI_MISO: J1.13 (Pin_13), U4.13 (MISO)
- new net SPI_MOSI: J1.17 (Pin_17), U4.14 (MOSI)
- new net SPI_SCK: J1.19 (Pin_19), U4.12 (SCK)
- new net SW: U5.1 (SW), U5.2 (SW)
- no-connect marks 0 -> 15
Other:
- added sheet Power and GNSS support (pinkman-support.kicad_sch)
- note added: "1 MAINBOARD INTERFACE"
- note added: "2 BAROMETER / I2C 0x5C"
- note added: "3 IMU / I2C 0x6A"
- note added: "4 SHARED I2C PULL-UPS"
- note added: "5 GPS / UART + I2C 0x42"
- note added: "6 433 MHz LORA RADIO"
- note added: "7 5 V TO 3.3 V POWER"
- note added: "Connect the listed 433 MHz antenna to module IPEX. DIO0 = IRQ; DIO1 available for radio driver. Keep antenna and radio away from GNSS input."
- note added: "INT1 test point: high impedance at power-on. INT2 and NC pins intentionally open."
- note added: "Keep pressure port unobstructed. Configure DRDY polarity in firmware."
- note added: "One pair for barometer, IMU and GPS. Start at 100 kHz; confirm rise time on bench."
- note added: "Pin 5 = +24 V on mainboard: intentionally NC. Pin 10 unused. Logic signals are 3.3 V. Works in module slot A or B with matching firmware."
- note added: "Power parts, test points and antenna bias are on page 2. No +24 V connection on this module."
- note added: "Slot B: I2C = Wire1; SPI = SPI1; UART = Serial8 Slot A: I2C = Wire; SPI = SPI; UART = Serial7"
- note added: "VIO_SEL / SAFEBOOT_N / EXTINT / RESET_N open. V_BCKP open: cold start after power removal. PPS must remain high impedance at startup."
- title: (none) -> PINKMAN - Sensors, GNSS and LoRa

Commit message: Simplified Schematic
Parts:
- removed R1, R2: 4.7k, Resistor_SMD:R_0603_1608Metric, symbol Device:R
- added R10, R11, R12, R13, R14, R9: 4.7k, symbol Device:R
- renumbered U1 to Altimeter, U3 to GPS, U2 to IMU, U4 to Radio
Connections:
- net +3V3: now also R10.2, R11.2, R12.2, R13.2, R14.2, R9.1
- net I2C_SCL: now also R12.1, R13.1, R9.2
- net I2C_SDA: now also R10.1, R11.1, R14.1
Other:
- note removed: "1 MAINBOARD INTERFACE"
- note removed: "2 BAROMETER / I2C 0x5C"
- note removed: "3 IMU / I2C 0x6A"
- note removed: "4 SHARED I2C PULL-UPS"
- note removed: "5 GPS / UART + I2C 0x42"
- note removed: "6 433 MHz LORA RADIO"
- note removed: "7 5 V TO 3.3 V POWER"
- title: PINKMAN - Sensors, GNSS and LoRa -> PINKMAN 
