File: pinkman/pinkman.kicad_sch (KiCad schematic)
At the start: 7 parts, among them J1 TSM-110-01-T-DV

Commit message: ALT & IMU
Parts:
- removed Altimeter: LPS22DFTR, QFN_22DFTR_STM, symbol Pinkman Altimeter:LPS22DFTR
- removed GPS: MAX-M10M-00B, MOD18_MAX-M10M_UBL, symbol GPS:MAX-M10M-00B
- removed IMU: LSM6DSO32TR, LGA-14L_2P5X3X0P83_STM, symbol IMU:LSM6DSO32TR
- removed J1: TSM-110-01-T-DV, MDFC Common:CONN_TSM-110-01-T-DV_SAI, symbol MDFC Common:TSM-110-01-T-DV
- removed Radio: RA-02, RA-02_AIT, symbol Radio:RA-02
- removed Regulator: LTC3601EMSE-TRPBF, MSOP-16_MSE_LIT, symbol Regulator:LTC3601EMSE-TRPBF
- added Altimeter: LPS22DFTR, Pinkman Local:QFN_22DFTR_STM, symbol Pinkman Local:LPS22DFTR
- added C2, C3, C4, C5, C6, C8: 100nF, Capacitor_SMD:C_0603_1608Metric, symbol Device:C
- added C7, C9: 10uF, Capacitor_SMD:C_0805_2012Metric, symbol Device:C
- added GPS: MAX-M10M-00B, Pinkman Local:MOD18_MAX-M10M_UBL, symbol Pinkman Local:MAX-M10M-00B
- added IMU: LSM6DSO32TR, Pinkman Local:LGA-14L_2P5X3X0P83_STM, symbol Pinkman Local:LSM6DSO32TR
- added J1: TSM-110-01-T-DV, MDFC Common:CONN_TSM-110-01-T-DV_SAI, symbol Connector_Generic:Conn_02x10_Odd_Even
- added R10, R11, R12, R13, R14, R9: 4.7k, symbol Device:R
- added R3, R4: 10k, Resistor_SMD:R_0603_1608Metric, symbol Device:R
- added Radio: RA-02, Pinkman Local:RA-02_AIT, symbol Pinkman Local:RA-02
- added TP1: IMU_INT1, TestPoint:TestPoint_Pad_D1.5mm, symbol Connector:TestPoint
- added U5: LTC3601EMSE-TRPBF, Pinkman Local:MSOP-16_MSE_LIT, symbol Pinkman Local:LTC3601EMSE-TRPBF
- C1: value 100 nF -> 100nF; footprint (none) -> Capacitor_SMD:C_0603_1608Metric
Connections:
- net GND: now reaches C1.2
- net GND: now also Altimeter.3 (RES), Altimeter.5 (SDO/SA0), Altimeter.8 (GND_IO), Altimeter.9 (GND), C2.2, C3.2, C4.2, C5.2, C6.2, C7.2, C8.2, C9.2, GPS.1 (GND), GPS.10 (GND), GPS.12 (GND), IMU.1 (SDO/SA0), IMU.2 (SDx), IMU.3 (SCx), IMU.6 (GND), IMU.7 (GND), J1.1 (Pin_1), J1.2 (Pin_2), J1.3 (Pin_3), J1.4 (Pin_4), Radio.1 (GND), Radio.16 (GND), Radio.2 (GND), Radio.9 (GND), U5.15 (MODE/SYNC), U5.17 (EPAD), U5.3 (PGND), U5.4 (PGND)
- net Earth renamed +3V3
- net +3V3: now also Altimeter.1 (Vdd_IO), Altimeter.10 (VDD), Altimeter.6 (CS), C2.1, C3.1, C4.1, C5.1, C6.1, C7.1, C8.1, C9.1, GPS.7 (V_IO), GPS.8 (VCC), IMU.12 (CS), IMU.5 (VDDIO), IMU.8 (VDD), R10.2, R11.2, R12.2, R13.2, R14.2, R3.1, R4.1, R9.1, Radio.3 (3.3V), U5.7 (VON)
- new net +5V_IN: J1.7 (Pin_7), U5.12 (RUN), U5.13 (VIN), U5.14 (VIN)
- new net BARO_DRDY: Altimeter.7 (INT_DRDY), J1.20 (Pin_20)
- new net BOOST: U5.5 (BOOST)
- new net FB: U5.9 (FB)
- new net GNSS_RF: GPS.11 (RF_IN)
- new net GPS_PPS: GPS.4 (TIMEPULSE), J1.14 (Pin_14)
- new net GPS_VCC_RF: GPS.14 (VCC_RF)
- new net HOST_UART_RX: GPS.2 (TXD), J1.18 (Pin_18)
- new net HOST_UART_TX: GPS.3 (RXD), J1.16 (Pin_16)
- new net I2C_SCL: Altimeter.2 (SCL), GPS.17 (SCL), IMU.13 (SCL), J1.6 (Pin_6), R12.1, R13.1, R9.2
- new net I2C_SDA: Altimeter.4 (SDA/SDI/SDISDO), GPS.16 (SDA), IMU.14 (SDA), J1.8 (Pin_8), R10.1, R11.1, R14.1
- new net IMU_INT1: IMU.4 (INT1), TP1.1
- new net INTVCC: U5.10 (ITH), U5.6 (INTVCC), U5.8 (RT)
- new net POWER_GOOD: U5.16 (PGOOD)
- new net RADIO_DIO0: J1.15 (Pin_15), Radio.5 (DIO0)
- new net RADIO_DIO1: J1.12 (Pin_12), Radio.6 (DIO1)
- new net RADIO_RESET_N: J1.9 (Pin_9), R3.2, Radio.4 (RESET)
- new net SOFTSTART: U5.11 (TRACK)
- new net SPI_CS_N: J1.11 (Pin_11), R4.2, Radio.15 (NSS)
- new net SPI_MISO: J1.13 (Pin_13), Radio.13 (MISO)
- new net SPI_MOSI: J1.17 (Pin_17), Radio.14 (MOSI)
- new net SPI_SCK: J1.19 (Pin_19), Radio.12 (SCK)
- new net SW: U5.1 (SW), U5.2 (SW)
- no-connect marks 0 -> 15
Other:
- added sheet Power and GNSS support (pinkman-support.kicad_sch)
- note added: "Connect the listed 433 MHz antenna to module IPEX. DIO0 = IRQ; DIO1 available for radio driver. Keep antenna and radio away from GNSS input."
- note added: "INT1 test point: high impedance at power-on. INT2 and NC pins intentionally open."
- note added: "Keep pressure port unobstructed. Configure DRDY polarity in firmware."
- note added: "One pair for barometer, IMU and GPS. Start at 100 kHz; confirm rise time on bench."
- note added: "Pin 5 = +24 V on mainboard: intentionally NC. Pin 10 unused. Logic signals are 3.3 V. Works in module slot A or B with matching firmware."
- note added: "Power parts, test points and antenna bias are on page 2. No +24 V connection on this module."
- note added: "Slot B: I2C = Wire1; SPI = SPI1; UART = Serial8 Slot A: I2C = Wire; SPI = SPI; UART = Serial7"
- note added: "VIO_SEL / SAFEBOOT_N / EXTINT / RESET_N open. V_BCKP open: cold start after power removal. PPS must remain high impedance at startup."
- title: (none) -> PINKMAN 

Commit message: Near Finished
Parts:
- removed C6, C8: 100nF, Capacitor_SMD:C_0603_1608Metric, symbol Device:C
- removed C7, C9: 10uF, Capacitor_SMD:C_0805_2012Metric, symbol Device:C
- removed R11, R12, R13, R14: 4.7k, symbol Device:R
- removed R3, R4: 10k, Resistor_SMD:R_0603_1608Metric, symbol Device:R
- removed TP1: IMU_INT1, TestPoint:TestPoint_Pad_D1.5mm, symbol Connector:TestPoint
- added Cap, Cap1: 100 nF, Package_TO_SOT_SMD:TDSON-8-1, symbol Device:C
- added L3: 2.2 uH, Package_SON:VSON-10-1EP_3x3mm_P0.5mm_EP1.65x2.4mm, symbol Device:L
- added R1: 180k, Package_DIP:DIP-8_W7.62mm, symbol Device:R
- added R2: 40k, Package_DIP:DIP-8_W7.62mm, symbol Device:R
- C1: value 100nF -> 2.2 uF; footprint Capacitor_SMD:C_0603_1608Metric -> (none)
- C2: value 100nF -> 22 uF; footprint Capacitor_SMD:C_0603_1608Metric -> (none)
- C3: value 100nF -> 100 nF; footprint Capacitor_SMD:C_0603_1608Metric -> (none)
- C4, C5: value 100nF -> 10 pF; footprint Capacitor_SMD:C_0603_1608Metric -> (none)
- renumbered Altimeter to Barometer, U5 to Regulator
Connections:
- net +5V_IN is gone; now on net +5V: J1.7 (Pin_7), Regulator.12 (RUN), Regulator.13 (VIN), Regulator.14 (VIN)
- net GPS_VCC_RF is gone; now on net +5V: GPS.14 (VCC_RF)
- net POWER_GOOD is gone; now on net GND: Regulator.16 (PGOOD)
- net SOFTSTART is gone; now on net GND: Regulator.11 (TRACK)
- net BOOST: now also C3.1
- net FB: now also C4.2, R1.2, R2.1
- net GND: now also IMU.9 (INT2), Cap.2, Cap1.2, R2.2; no longer C3.2, C4.2, Regulator.15 (MODE/SYNC)
- net SW: now also C3.2, L3.1
- net UART_GPS_TX_1: now reaches J1.10 (Pin_10)
- net UART_GPS_TX_1: now also GPS.2 (TXD)
- net +24V: now reaches J1.5 (Pin_5)
- net GPS_EXTINT_1: now reaches GPS.5 (EXTINT)
- net GPS_EXTINT_1: now also J1.13 (Pin_13)
- net +5V: now reaches GPS.6 (V_BCKP)
- net +5V: now also C2.1, GPS.7 (V_IO), GPS.8 (VCC)
- net +3V3 renamed +3.3V
- net +3.3V: now also Cap.1, Cap1.1, L3.2, R1.1; no longer Barometer.6 (CS), C1.1, C2.1, C3.1, GPS.7 (V_IO), GPS.8 (VCC), IMU.12 (CS)
- net BARO_DRDY renamed I2C_Baro_DRDY_1
- net I2C_Baro_DRDY_1: now also J1.16 (Pin_16); no longer J1.20 (Pin_20)
- net GNSS_RF: no longer names the net of GPS.11 (RF_IN)
- net GPS_PPS renamed GPS_PPS_1
- net HOST_UART_RX: no longer names the net of J1.18 (Pin_18)
- net HOST_UART_RX: no longer GPS.2 (TXD)
- net HOST_UART_TX renamed UART_GPS_RX_1
- net UART_GPS_RX_1: now also J1.12 (Pin_12); no longer J1.16 (Pin_16)
- net IMU_INT1 renamed I2C_IMU_DRDY_1
- net I2C_IMU_DRDY_1: now also J1.15 (Pin_15)
- net INTVCC renamed Cap2GND
- net Cap2GND: now also C1.1, Regulator.15 (MODE/SYNC)
- net RADIO_DIO0: no longer names the net of Radio.5 (DIO0)
- net RADIO_DIO0: no longer J1.15 (Pin_15)
- net RADIO_DIO1: no longer names the net of Radio.6 (DIO1)
- net RADIO_DIO1: no longer J1.12 (Pin_12)
- net RADIO_RESET_N renamed Radio_Reset_1
- net Radio_Reset_1: no longer J1.9 (Pin_9)
- net SPI_CS_N renamed SPI_LoRa_MISO_1
- net SPI_LoRa_MISO_1: now also Radio.13 (MISO); no longer Radio.15 (NSS)
- removed net SPI_MISO: J1.13 (Pin_13), Radio.13 (MISO)
- net SPI_MOSI renamed I2C_IMU_CS_0
- net I2C_IMU_CS_0: no longer Radio.14 (MOSI)
- net SPI_SCK renamed SPI_LoRa_SCK_1
- new net I2C_Baro_CS_1: Barometer.6 (CS)
- new net I2C_IMU_CS_1: IMU.12 (CS)
- new net SPI_LoRa_MOSI_1: J1.9 (Pin_9), Radio.14 (MOSI)
- new net SPI_LoRa_NSS_1: J1.20 (Pin_20), Radio.15 (NSS)
- no-connect marks 15 -> 0
Other:
- removed sheet Power and GNSS support
- note removed: "Connect the listed 433 MHz antenna to module IPEX. DIO0 = IRQ; DIO1 available for radio driver. Keep antenna and radio away from GNSS input."
- note removed: "INT1 test point: high impedance at power-on. INT2 and NC pins intentionally open."
- note removed: "Keep pressure port unobstructed. Configure DRDY polarity in firmware."
- note removed: "One pair for barometer, IMU and GPS. Start at 100 kHz; confirm rise time on bench."
- note removed: "Pin 5 = +24 V on mainboard: intentionally NC. Pin 10 unused. Logic signals are 3.3 V. Works in module slot A or B with matching firmware."
- note removed: "Power parts, test points and antenna bias are on page 2. No +24 V connection on this module."
- note removed: "Slot B: I2C = Wire1; SPI = SPI1; UART = Serial8 Slot A: I2C = Wire; SPI = SPI; UART = Serial7"
- note removed: "VIO_SEL / SAFEBOOT_N / EXTINT / RESET_N open. V_BCKP open: cold start after power removal. PPS must remain high impedance at startup."
- moved on the sheet: Regulator
