File: heisenberg/heisenberg.kicad_pcb (KiCad board)
At the start: 2 copper layers, 117 x 63.5 mm, 19 parts, among them J1 HLE-110-02-L-DV-BE-K-TR, J2 HLE-110-02-L-DV-BE-K-TR, J3 TSM-108-01-F-DV, J4 S16B-XH-A, U1 Teensy4.1

Commit message: Created Tuco board outline, heisenberg pin labels
Other:
- copper layers 2 -> 4
- board text added: "+5V GND +3V3 GND"
- board text added: "GND +3V3"
- board text added: "GRN2B GRN1B RED2B RED1B YEL2B YEL1B BLU2B BLU1B ORN5B"
- board text added: "ORN2B ORN4B ORN1B ORN3B ORN5B"
- board text added: "PWR10 PWR9 RED2A RED1A GRN2A GRN1A ORN3A YEL2A YEL1A ORN2A ORN1A"
- board text added: "SERVO8 SERVO9 SERVO10 SERVO11 SERVO12 SERVO13 SERVO14 PURP1A ORN3A ORN4A PWR1 PWR2 BLU1A BLU2A SERVO6 SERVO7 PWR5"

Commit message: Main board MOD A&B pins & routing
V1 of  the initial module A & B routing so other people can have a starting point for their pin layout

dont mind the naming scheme i need to fix that
Parts:
- removed REF** (x4): MountingHole_3.2mm_M3, MountingHole:MountingHole_3.2mm_M3
- removed REF** (x8): MountingHole_2.2mm_M2, MountingHole:MountingHole_2.2mm_M2
- removed REF**: ESD-Logo_6.6x6mm_SilkScreen, Symbol:ESD-Logo_6.6x6mm_SilkScreen
Connections:
- J1 pad 01: unconnected-(J1-Pad01) -> +5V
- J1 pad 02: unconnected-(J1-Pad02) -> GND
- J1 pad 03: unconnected-(J1-Pad03) -> +24V
- J1 pad 04: unconnected-(J1-Pad04) -> GND
- J1 pad 05: unconnected-(J1-Pad05) -> GND
- J1 pad 06: unconnected-(J1-Pad06) -> /PWM_CS_A
- J1 pad 07: unconnected-(J1-Pad07) -> GND
- J1 pad 08: unconnected-(J1-Pad08) -> /SPI_A_CS
- J1 pad 09: unconnected-(J1-Pad09) -> /UART_A_TX7
- J1 pad 10: unconnected-(J1-Pad10) -> /A14_A
- J1 pad 11: unconnected-(J1-Pad11) -> /UART_A_RX7
- J1 pad 12: unconnected-(J1-Pad12) -> /SPI_A_SCK
- J1 pad 13: unconnected-(J1-Pad13) -> /SPI_A_MISO
- J1 pad 14: unconnected-(J1-Pad14) -> /A0_TX
- J1 pad 15: unconnected-(J1-Pad15) -> /SPI_A_MOSI
- J1 pad 16: unconnected-(J1-Pad16) -> /I2C_A_SCL
- J1 pad 17: unconnected-(J1-Pad17) -> /PWM_A
- J1 pad 18: unconnected-(J1-Pad18) -> /I2C_A_SDA
- J1 pad 19: unconnected-(J1-Pad19) -> /A15_A
- J1 pad 20: unconnected-(J1-Pad20) -> /A1_RX
- J2 pad 01: unconnected-(J2-Pad01) -> /A17_B
- J2 pad 02: unconnected-(J2-Pad02) -> /I2C_B_SCL
- J2 pad 03: unconnected-(J2-Pad03) -> /SPI_B_CS1
- J2 pad 04: unconnected-(J2-Pad04) -> /I2C_B_SDA
- J2 pad 05: unconnected-(J2-Pad05) -> /SPI_B_MISO1
- J2 pad 06: unconnected-(J2-Pad06) -> /A7_RX5
- J2 pad 07: unconnected-(J2-Pad07) -> /PWM1_B
- J2 pad 08: unconnected-(J2-Pad08) -> /A6_TX5
- J2 pad 09: unconnected-(J2-Pad09) -> /SPI_B_MOSI1
- J2 pad 10: unconnected-(J2-Pad10) -> /A16_B
- J2 pad 11: unconnected-(J2-Pad11) -> /SPI_B_SCK1
- J2 pad 12: unconnected-(J2-Pad12) -> /TX8
- J2 pad 13: unconnected-(J2-Pad13) -> GND
- J2 pad 14: unconnected-(J2-Pad14) -> /RX8
- J2 pad 15: unconnected-(J2-Pad15) -> GND
- J2 pad 16: unconnected-(J2-Pad16) -> /PWM_B
- J2 pad 17: unconnected-(J2-Pad17) -> +24V
- J2 pad 18: unconnected-(J2-Pad18) -> GND
- J2 pad 19: unconnected-(J2-Pad19) -> +5V
- J2 pad 20: unconnected-(J2-Pad20) -> GND
- J3 pad 1: unconnected-(J3-Pad1) -> GND
- J3 pad 10: unconnected-(J3-Pad10) -> +24V
- J3 pad 11: unconnected-(J3-Pad11) -> GND
- J3 pad 12: unconnected-(J3-Pad12) -> /V_servo
- J3 pad 13: unconnected-(J3-Pad13) -> GND
- J3 pad 14: unconnected-(J3-Pad14) -> /V_servo
- J3 pad 15: unconnected-(J3-Pad15) -> GND
- J3 pad 16: unconnected-(J3-Pad16) -> /V_servo
- J3 pad 2: unconnected-(J3-Pad2) -> GND
- J3 pad 3: unconnected-(J3-Pad3) -> +5V
- J3 pad 4: unconnected-(J3-Pad4) -> +5V
- J3 pad 5: unconnected-(J3-Pad5) -> /GPIO_PWR
- J3 pad 6: unconnected-(J3-Pad6) -> /A_RX6_SDA2_PWM
- J3 pad 7: unconnected-(J3-Pad7) -> /A_CTX1_PWM
- J3 pad 8: unconnected-(J3-Pad8) -> /A_TX6_SCL2_PWM
- J3 pad 9: unconnected-(J3-Pad9) -> /A_CRX1_PWM
- J4 pad 1: unconnected-(J4-Pad1) -> GND
- J4 pad 10: unconnected-(J4-Pad10) -> /PWM_TX2
- J4 pad 11: unconnected-(J4-Pad11) -> /PWM_5
- J4 pad 12: unconnected-(J4-Pad12) -> /PWM_4
- J4 pad 13: unconnected-(J4-Pad13) -> /PWM_3
- J4 pad 14: unconnected-(J4-Pad14) -> /PWM_2
- J4 pad 15: unconnected-(J4-Pad15) -> /PWM_1
- J4 pad 16: unconnected-(J4-Pad16) -> +5V
- J4 pad 2: unconnected-(J4-Pad2) -> /V_servo
- J4 pad 3: unconnected-(J4-Pad3) -> GND
- J4 pad 4: unconnected-(J4-Pad4) -> /V_servo
- J4 pad 5: unconnected-(J4-Pad5) -> GND
- J4 pad 6: unconnected-(J4-Pad6) -> /V_servo
- J4 pad 7: unconnected-(J4-Pad7) -> /CAN_Servo_CTX3
- J4 pad 8: unconnected-(J4-Pad8) -> /CAN_Servo_CRX3
- J4 pad 9: unconnected-(J4-Pad9) -> /PWM_RX2
- U1 pad 10: unconnected-(U1-8_TX2_IN1-Pad10) -> /PWM_RX2
- U1 pad 11: unconnected-(U1-9_OUT1C-Pad11) -> /PWM_A
- U1 pad 12: unconnected-(U1-10_CS_MQSR-Pad12) -> /PWM1_B
- U1 pad 13: unconnected-(U1-11_MOSI_CTX1-Pad13) -> /SPI_A_MOSI
- U1 pad 14: unconnected-(U1-12_MISO_MQSL-Pad14) -> /SPI_A_MISO
- U1 pad 16: unconnected-(U1-24_A10_TX6_SCL2-Pad16) -> /A_TX6_SCL2_PWM
- U1 pad 17: unconnected-(U1-25_A11_RX6_SDA2-Pad17) -> /A_RX6_SDA2_PWM
- U1 pad 18: unconnected-(U1-26_A12_MOSI1-Pad18) -> /SPI_B_MOSI1
- U1 pad 19: unconnected-(U1-27_A13_SCK1-Pad19) -> /SPI_B_SCK1
- U1 pad 2: unconnected-(U1-0_RX1_CRX2_CS1-Pad2) -> /SPI_B_CS1
- U1 pad 20: unconnected-(U1-28_RX7-Pad20) -> /UART_A_RX7
- U1 pad 21: unconnected-(U1-29_TX7-Pad21) -> /UART_A_TX7
- U1 pad 22: unconnected-(U1-30_CRX3-Pad22) -> /CAN_Servo_CRX3
- U1 pad 23: unconnected-(U1-31_CTX3-Pad23) -> /CAN_Servo_CTX3
- U1 pad 24: unconnected-(U1-32_OUT1B-Pad24) -> /GPIO_PWR
- U1 pad 25: unconnected-(U1-33_MCLK2-Pad25) -> /PWM_B
- U1 pad 26: unconnected-(U1-34_RX8-Pad26) -> /RX8
- U1 pad 27: unconnected-(U1-35_TX8-Pad27) -> /TX8
- U1 pad 28: unconnected-(U1-36_CS-Pad28) -> /PWM_CS_A
- U1 pad 29: unconnected-(U1-37_CS-Pad29) -> /SPI_A_CS
- U1 pad 3: unconnected-(U1-1_TX1_CTX2_MISO1-Pad3) -> /SPI_B_MISO1
- U1 pad 30: unconnected-(U1-38_CS1_IN1-Pad30) -> /A14_A
- U1 pad 31: unconnected-(U1-39_MISO1_OUT1A-Pad31) -> /A15_A
- U1 pad 32: unconnected-(U1-40_A16-Pad32) -> /A16_B
- U1 pad 33: unconnected-(U1-41_A17-Pad33) -> /A17_B
- U1 pad 35: unconnected-(U1-13_SCK_LED-Pad35) -> /SPI_A_SCK
- U1 pad 36: unconnected-(U1-14_A0_TX3_SPDIF_OUT-Pad36) -> /A0_TX
- U1 pad 37: unconnected-(U1-15_A1_RX3_SPDIF_IN-Pad37) -> /A1_RX
- U1 pad 38: unconnected-(U1-16_A2_RX4_SCL1-Pad38) -> /I2C_B_SCL
- U1 pad 39: unconnected-(U1-17_A3_TX4_SDA1-Pad39) -> /I2C_B_SDA
- U1 pad 4: unconnected-(U1-2_OUT2-Pad4) -> /PWM_1
- U1 pad 40: unconnected-(U1-18_A4_SDA-Pad40) -> /I2C_A_SDA
- U1 pad 41: unconnected-(U1-19_A5_SCL-Pad41) -> /I2C_A_SCL
- U1 pad 42: unconnected-(U1-20_A6_TX5_LRCLK1-Pad42) -> /A6_TX5
- U1 pad 43: unconnected-(U1-21_A7_RX5_BCLK1-Pad43) -> /A7_RX5
- U1 pad 44: unconnected-(U1-22_A8_CTX1-Pad44) -> /A_CTX1_PWM
- U1 pad 45: unconnected-(U1-23_A9_CRX1_MCLK1-Pad45) -> /A_CRX1_PWM
- U1 pad 5: unconnected-(U1-3_LRCLK2-Pad5) -> /PWM_2
- U1 pad 6: unconnected-(U1-4_BCLK2-Pad6) -> /PWM_3
- U1 pad 7: unconnected-(U1-5_IN2-Pad7) -> /PWM_4
- U1 pad 8: unconnected-(U1-6_OUT1D-Pad8) -> /PWM_5
- U1 pad 9: unconnected-(U1-7_RX2_OUT1A-Pad9) -> /PWM_TX2
Routing:
- net /PWM_B: track 0.00 -> 140.5 mm
- net /RX8: track 0.00 -> 134.1 mm
- net /PWM_CS_A: track 0.00 -> 131.5 mm
- net /TX8: track 0.00 -> 127.5 mm
- net /SPI_A_CS: track 0.00 -> 124.8 mm
- net /A14_A: track 0.00 -> 118.0 mm
- net /A16_B: track 0.00 -> 108.2 mm
- net /SPI_A_SCK: track 0.00 -> 100.6 mm
- net /A0_TX: track 0.00 -> 93.0 mm
- net /PWM_1: track 0.00 -> 91.6 mm
- net /PWM_2: track 0.00 -> 88.1 mm
- net /PWM_3: track 0.00 -> 84.5 mm
- net /PWM_4: track 0.00 -> 81.0 mm
- net /A6_TX5: track 0.00 -> 78.6 mm
- net /PWM_5: track 0.00 -> 77.4 mm
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Other:
- board text added: "Rev.0 2026 Matthew Saintilus"
- board text removed: "Rev.0 2026 Matthew Santilius"

Commit message: attempt number 2 at routing
This time they are identical schematic layout for A & B and i used the 4 layers to route to potential via points b4 connection
Connections:
- J1 pad 01: +5V -> GND
- J1 pad 03: +24V -> GND
- J1 pad 05: GND -> +24V
- J1 pad 06: /PWM_CS_A -> /I2C_A_SCL
- J1 pad 07: GND -> +5V
- J1 pad 08: /SPI_A_CS -> /I2C_A_SDA
- J1 pad 09: /UART_A_TX7 -> /A15_A
- J1 pad 10: /A14_A -> /A1_RX
- J1 pad 11: /UART_A_RX7 -> /SPI_A_CS
- J1 pad 12: /SPI_A_SCK -> /A0_TX
- J1 pad 14: /A0_TX -> /A14_A
- J1 pad 15: /SPI_A_MOSI -> /PWM_A
- J1 pad 16: /I2C_A_SCL -> /UART_A_TX7
- J1 pad 17: /PWM_A -> /SPI_A_MOSI
- J1 pad 18: /I2C_A_SDA -> /UART_A_RX7
- J1 pad 19: /A15_A -> /SPI_A_SCK
- J1 pad 20: /A1_RX -> /PWM_CS_A
- J2 pad 01: /A17_B -> GND
- J2 pad 02: /I2C_B_SCL -> GND
- J2 pad 03: /SPI_B_CS1 -> GND
- J2 pad 04: /I2C_B_SDA -> GND
- J2 pad 05: /SPI_B_MISO1 -> +24V
- J2 pad 06: /A7_RX5 -> /I2C_B_SCL
- J2 pad 07: /PWM1_B -> +5V
- J2 pad 08: /A6_TX5 -> /I2C_B_SDA
- J2 pad 09: /SPI_B_MOSI1 -> /A17_B
- J2 pad 10: /A16_B -> /A7_RX5
- J2 pad 11: /SPI_B_SCK1 -> /SPI_B_CS1
- J2 pad 12: /TX8 -> /A6_TX5
- J2 pad 13: GND -> /SPI_B_MISO1
- J2 pad 14: /RX8 -> /A16_B
- J2 pad 15: GND -> /PWM_B
- J2 pad 16: /PWM_B -> /UART_B_TX8
- J2 pad 17: +24V -> /SPI_B_MOSI1
- J2 pad 18: GND -> /UART_B_RX8
- J2 pad 19: +5V -> /SPI_B_SCK1
- J2 pad 20: GND -> /PWM1_B
- U1 pad 26: /RX8 -> /UART_B_RX8
- U1 pad 27: /TX8 -> /UART_B_TX8
Routing:
- net /UART_B_RX8: track 0.00 -> 134.3 mm
- net /RX8: track 134.1 -> 0.00 mm
- net /TX8: track 127.5 -> 0.00 mm
- net /UART_B_TX8: track 0.00 -> 125.4 mm
- net /PWM_CS_A: track 131.5 -> 81.9 mm
- net /PWM1_B: track 48.8 -> 93.7 mm
- net /SPI_A_CS: track 124.8 -> 86.4 mm
- net /SPI_A_SCK: track 100.6 -> 62.7 mm
- net /PWM_B: track 140.5 -> 106.4 mm
- net /I2C_A_SDA: track 63.1 -> 91.6 mm
- net /I2C_A_SCL: track 67.8 -> 91.7 mm
- net /UART_A_TX7: track 72.3 -> 94.3 mm
- net /UART_A_RX7: track 68.8 -> 87.5 mm
- net /A14_A: track 118.0 -> 104.5 mm
- net /I2C_B_SCL: track 62.9 -> 74.9 mm
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
Commit message: V2 pin layout main board
Rerouted the wiring to the conectors on the main board in a better less cluttered way all that it needs is vias b4 connecting
Connections:
- J1 pad 09: /A15_A -> /PWM_CS_A
- J1 pad 20: /PWM_CS_A -> /A15_A
- J2 pad 09: /A17_B -> /PWM1_B
- J2 pad 20: /PWM1_B -> /A17_B
Routing:
- net /PWM1_B: track 93.7 -> 0.00 mm
- net /A17_B: track 77.6 -> 120.0 mm
- net /A1_RX: track 74.7 -> 97.2 mm
- net /A16_B: track 115.9 -> 102.5 mm
- net /A15_A: track 79.4 -> 74.0 mm
- net /I2C_B_SDA: track 79.0 -> 73.7 mm
- net /PWM_CS_A: track 81.9 -> 86.9 mm
- net /UART_B_TX8: track 125.4 -> 129.9 mm
- net /UART_A_TX7: track 94.3 -> 90.0 mm
- net /I2C_A_SDA: track 91.6 -> 87.4 mm
- net /UART_A_RX7: track 87.5 -> 83.8 mm
- net /SPI_A_SCK: track 62.7 -> 65.5 mm
- net /A6_TX5: track 79.1 -> 81.8 mm
- net /SPI_A_CS: track 86.4 -> 88.7 mm
- net /I2C_B_SCL: track 74.9 -> 72.8 mm
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
Commit message: Addition to the V2 reroute update
there was a unconnected pin and i untangled 1 route
Routing:
- net /PWM1_B: track 0.00 -> 45.6 mm
- net /PWM_CS_A: track 86.9 -> 90.8 mm
- net /SPI_A_CS: track 88.7 -> 85.6 mm

Commit message: updated power pins layouot
apparently this was never pusheded
Connections:
- J3 pad 1: GND -> /GPIO_PWR
- J3 pad 10: +24V -> +5V
- J3 pad 2: GND -> /A_RX6_SDA2_PWM
- J3 pad 3: +5V -> /A_CTX1_PWM
- J3 pad 4: +5V -> /A_TX6_SCL2_PWM
- J3 pad 5: /GPIO_PWR -> /A_CRX1_PWM
- J3 pad 6: /A_RX6_SDA2_PWM -> GND
- J3 pad 7: /A_CTX1_PWM -> +5V
- J3 pad 8: /A_TX6_SCL2_PWM -> +24V
- J3 pad 9: /A_CRX1_PWM -> GND
Routing:
- net +5V: track 0.00 -> 99.6 mm
- net +24V: track 0.00 -> 99.2 mm
- net /A_CRX1_PWM: track 0.00 -> 68.2 mm
- net /A_CTX1_PWM: track 0.00 -> 62.2 mm
- net /A_TX6_SCL2_PWM: track 0.00 -> 31.8 mm
- net /A_RX6_SDA2_PWM: track 0.00 -> 25.9 mm
- net /GPIO_PWR: track 0.00 -> 11.0 mm
- net GND: track 0.00 -> 1.21 mm
Changed lines of the file:
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@@
 			(size 1.27 3.683)
 			(layers "F.Cu" "F.Mask" "F.Paste")
-			(net "GND")
+			(net "/GPIO_PWR")
 			(pinfunction "1_1")
 			(pintype "unspecified")
@@
 			(size 1.27 3.683)
 			(layers "F.Cu" "F.Mask" "F.Paste")
-			(net "GND")
+			(net "/A_RX6_SDA2_PWM")
 			(pinfunction "2_2")
 			(pintype "unspecified")
@@
 			(size 1.27 3.683)
 			(layers "F.Cu" "F.Mask" "F.Paste")
-			(net "+5V")
+			(net "/A_CTX1_PWM")
 			(pinfunction "3_3")
 			(pintype "unspecified")
@@
 			(size 1.27 3.683)
 			(layers "F.Cu" "F.Mask" "F.Paste")
-			(net "+5V")
+			(net "/A_TX6_SCL2_PWM")
 			(pinfunction "4_4")
 			(pintype "unspecified")
@@
 			(size 1.27 3.683)
 			(layers "F.Cu" "F.Mask" "F.Paste")
-			(net "/GPIO_PWR")
+			(net "/A_CRX1_PWM")
 			(pinfunction "5_5")
 			(pintype "unspecified")
@@
 			(size 1.27 3.683)
 			(layers "F.Cu" "F.Mask" "F.Paste")
-			(net "/A_RX6_SDA2_PWM")
+			(net "GND")
 			(pinfunction "6_6")
 			(pintype "unspecified")
@@
 			(size 1.27 3.683)
 			(layers "F.Cu" "F.Mask" "F.Paste")
-			(net "/A_CTX1_PWM")
+			(net "+5V")
 			(pinfunction "7_7")
 			(pintype "unspecified")
@@
 			(size 1.27 3.683)
 			(layers "F.Cu" "F.Mask" "F.Paste")
-			(net "/A_TX6_SCL2_PWM")
+			(net "+24V")
 			(pinfunction "8_8")
 			(pintype "unspecified")
@@
 			(size 1.27 3.683)
 			(layers "F.Cu" "F.Mask" "F.Paste")
-			(net "/A_CRX1_PWM")
+			(net "GND")
 			(pinfunction "9_9")
 			(pintype "unspecified")
@@
 			(size 1.27 3.683)
 			(layers "F.Cu" "F.Mask" "F.Paste")
-			(net "+24V")
+			(net "+5V")
 			(pinfunction "10_10")
 			(pintype "unspecified")
@@
 	)
 	(segment
+		(start 112.77 68.9765)
+		(end 112.77 70.183)
+		(width 0.2)
+		(layer "F.Cu")
+		(net "GND")
+	)
+	(segment
 		(start 122 55)
 		(end 126 55)
@@
 	)
 	(segment
+		(start 108.625 67.3715)
+		(end 108.625 60.875)
+		(width 0.2)
+		(layer "F.Cu")
+		(net "+5V")
+	)
+	(segment
+		(start 110.23 68.9765)
+		(end 108.625 67.3715)
+		(width 0.2)
+		(layer "F.Cu")
+		(net "+5V")
+	)
+	(segment
+		(start 78.94 31.19)
+		(end 31.245 31.19)
+		(width 0.2)
+		(layer "F.Cu")
+		(net "+5V")
+	)
+	(segment
+		(start 108.625 60.875)
+		(end 78.94 31.19)
+		(width 0.2)
+		(layer "F.Cu")
+		(net "+5V")
+	)
+	(segment
+		(start 110.23 68.9765)
+		(end 110.23 70.183)
+		(width 0.2)
+		(layer "F.Cu")
+		(net "+5V")
+	)
+	(segment
+		(start 102.61 68.9765)
+		(end 99.71 66.0765)
+		(width 0.2)
+		(layer "F.Cu")
+		(net "/GPIO_PWR")
+	)
+	(segment
+		(start 99.71 66.0765)
+		(end 99.71 59.1984)
+		(width 0.2)
+		(layer "F.Cu")
+		(net "/GPIO_PWR")
+	)
+	(segment
+		(start 102.5 64)
+		(end 102.5 64.75)
+		(width 0.2)
+		(layer "B.Cu")
+		(net "/A_RX6_SDA2_PWM")
+	)
+	(segment
+		(start 88.7316 66)
+		(end 81.93 59.1984)
+		(width 0.2)
+		(layer "B.Cu")
+		(net "/A_RX6_SDA2_PWM")
+	)
+	(segment
+		(start 102.5 64.75)
+		(end 101.25 66)
+		(width 0.2)
+		(layer "B.Cu")
+		(net "/A_RX6_SDA2_PWM")
+	)
+	(segment
+		(start 101.25 66)
+		(end 88.7316 66)
+		(width 0.2)
+		(layer "B.Cu")
+		(net "/A_RX6_SDA2_PWM")
+	)
+	(segment
+		(start 107.69 64.0235)
+		(end 107.69 65.23)
+		(width 0.2)
+		(layer "B.Cu")
+		(net "/A_RX6_SDA2_PWM")
+	)
+	(segment
+		(start 52 76.5)
+		(end 51.45 75.95)
+		(width 0.2)
+		(layer "F.Cu")
+		(net "/A_CTX1_PWM")
+	)
+	(segment
+		(start 51.45 75.95)
+		(end 51.45 74.4384)
+		(width 0.2)
+		(layer "F.Cu")
+		(net "/A_CTX1_PWM")
+	)
+	(segment
+		(start 105.15 75.263)
+		(end 105.15 68.9765)
+		(width 0.2)
+		(layer "F.Cu")
+		(net "/A_CTX1_PWM")
+	)
+	(segment
+		(start 103.913 76.5)
+		(end 105.15 75.263)
+		(width 0.2)
+		(layer "F.Cu")
+		(net "/A_CTX1_PWM")
+	)
+	(segment
+		(start 103.913 76.5)
+		(end 52 76.5)
+		(width 0.2)
+		(layer "F.Cu")
+		(net "/A_CTX1_PWM")
+	)
+	(segment
+		(start 105.25 64)
+		(end 105.25 65)
+		(width 0.2)
+		(layer "B.Cu")
+		(net "/A_TX6_SCL2_PWM")
+	)
+	(segment
+		(start 86.7566 66.565)
+		(end 79.39 59.1984)
+		(width 0.2)
+		(layer "B.Cu")
+		(net "/A_TX6_SCL2_PWM")
+	)
+	(segment
+		(start 110.23 64.0235)
+		(end 110.23 65.23)
+		(width 0.2)
+		(layer "B.Cu")
+		(net "/A_TX6_SCL2_PWM")
+	)
+	(segment
+		(start 105.25 65)
+		(end 103.685 66.565)
+		(width 0.2)
+		(layer "B.Cu")
+		(net "/A_TX6_SCL2_PWM")
+	)
+	(segment
+		(start 103.685 66.565)
+		(end 86.7566 66.565)
+		(width 0.2)
+		(layer "B.Cu")
+		(net "/A_TX6_SCL2_PWM")
+	)
+	(segment
+		(start 48.91 76.41)
+		(end 48.91 74.4384)
+		(width 0.2)
+		(layer "F.Cu")
+		(net "/A_CRX1_PWM")
+	)
+	(segment
+		(start 105.203 77.75)
+		(end 107.69 75.263)
+		(width 0.2)
+		(layer "F.Cu")
+		(net "/A_CRX1_PWM")
+	)
+	(segment
+		(start 107.69 75.263)
+		(end 107.69 69.3765)
+		(width 0.2)
+		(layer "F.Cu")
+		(net "/A_CRX1_PWM")
+	)
+	(segment
+		(start 50.25 77.75)
+		(end 48.91 76.41)
+		(width 0.2)
+		(layer "F.Cu")
+		(net "/A_CRX1_PWM")
+	)
+	(segment
+		(start 105.203 77.75)
+		(end 50.25 77.75)
+		(width 0.2)
+		(layer "F.Cu")
+		(net "/A_CRX1_PWM")
+	)
+	(segment
+		(start 84.4 28.65)
+		(end 31.245 28.65)
+		(width 0.2)
+		(layer "F.Cu")
+		(net "+24V")
+	)
+	(segment
+		(start 110.23 54.48)
+		(end 84.4 28.65)
+		(width 0.2)
+		(layer "F.Cu")
+		(net "+24V")
+	)
+	(segment
+		(start 110.23 64.0235)
+		(end 110.23 54.48)
+		(width 0.2)
+		(layer "F.Cu")
+		(net "+24V")
+	)
+	(segment
