File: fring/fring.kicad_pcb (KiCad board)
At the start: 2 copper layers, 100 x 21.5 mm, 9 parts, among them J1 HLE-108-02-L-DV-K, J2 Conn_02x03_Odd_Even, J3 WE-RJ45_7499111447

Commit message: 90 percent done schematic
Parts:
- added U2: POE_Regulator_AG9924-MT, MDFC Common:AG9924-MT_SLV, F.Cu at (81.8, 89.4)
- added U5: Diode_PDS360-13, Fring Local:Diode_PDS360-13_DIO, F.Cu at (52.0, 75.0)
